File: flightcontroller.kicad_pcb (KiCad board)
At the start: 4 copper layers, 70 x 100 mm, 132 parts, among them J1 Conn_01x05_Pin, J10 Conn_01x03, J11 Conn_01x03, J12 Conn_01x03, J13 Conn_01x03, J14 Conn_01x03, J15 Conn_01x03, J16 Conn_01x03, J17 RC_USART2_3V3_LOGIC, J18 GPS, J19 TELEMETRY, J2 USB_C_Receptacle_USB2.0_14P, J20 COMPASS_I2C4_3V3, J21 AIRSPEED_I2C4_3V3, J22 SERVO_BEC_6V_INPUT, J23 BATTERY_SENSE_ONLY, J24 ACTIVE_BUZZER_5V_20mA_MAX, J3 Micro_SD_Card, J4 5V_REGULATED_INPUT, J5 Conn_01x03, J6 Conn_01x03, J7 Conn_01x03, J8 Conn_01x03, J9 Conn_01x03, Q1 MMBT3904, SW1 RESET, SW2 SAFETY, U1 STM32H743VITx, U2 ICM-42688-P, U3 ICM-42688-P, U4 BMI088, U5 MB85RS64, U6 BMP390, U7 BMP390, U8 TPS62162DSG, U9 USBLC6-2SC6, Y1 8MHz

Commit message: Update JST-GH interfaces and add board 3D preview
Parts:
- J1: value Conn_01x05_Pin -> SWD_CUSTOM_GH5; footprint Connector_PinHeader_2.54mm:PinHeader_1x05_P2.54mm_Vertical -> Connector_JST:JST_GH_SM05B-GHS-TB_1x05-1MP_P1.25mm_Horizontal
- J17: value RC_USART2_3V3_LOGIC -> RC_UART_GH6_NO_FLOW; footprint Connector_PinHeader_2.54mm:PinHeader_1x04_P2.54mm_Vertical -> Connector_JST:JST_GH_SM06B-GHS-TB_1x06-1MP_P1.25mm_Horizontal
- J18: value GPS -> GPS_PIXHAWK_GPS2; footprint Connector_PinHeader_2.54mm:PinHeader_1x04_P2.54mm_Vertical -> Connector_JST:JST_GH_SM06B-GHS-TB_1x06-1MP_P1.25mm_Horizontal
- J19: value TELEMETRY -> TELEM_GH6_NO_FLOW; footprint Connector_PinHeader_2.54mm:PinHeader_1x04_P2.54mm_Vertical -> Connector_JST:JST_GH_SM06B-GHS-TB_1x06-1MP_P1.25mm_Horizontal
- J20: value COMPASS_I2C4_3V3 -> COMPASS_I2C4_5V; footprint Connector_PinHeader_2.54mm:PinHeader_1x04_P2.54mm_Vertical -> Connector_JST:JST_GH_SM04B-GHS-TB_1x04-1MP_P1.25mm_Horizontal
- J21: value AIRSPEED_I2C4_3V3 -> AIRSPEED_I2C4_5V; footprint Connector_PinHeader_2.54mm:PinHeader_1x04_P2.54mm_Vertical -> Connector_JST:JST_GH_SM04B-GHS-TB_1x04-1MP_P1.25mm_Horizontal
- J24: value ACTIVE_BUZZER_5V_20mA_MAX -> BUZZER_5V_20mA_MAX; footprint Connector_PinHeader_2.54mm:PinHeader_1x02_P2.54mm_Vertical -> Connector_JST:JST_GH_SM02B-GHS-TB_1x02-1MP_P1.25mm_Horizontal
- moved J24 17.6 mm to (144.7, 151.5), turned to 90 degrees
- moved J1 5.13 mm to (81.3, 81.1), turned to -90 degrees
- moved J17 3.87 mm to (81.3, 106.8), turned to -90 degrees
- moved J18 3.87 mm to (81.3, 120.8), turned to -90 degrees
- moved J19 3.87 mm to (81.3, 134.8), turned to -90 degrees
- moved J20 3.82 mm to (90.8, 71.8), turned to 180 degrees
- moved J21 3.82 mm to (130.8, 71.8), turned to 180 degrees
Connections:
- J17 pad 4: GND -> unconnected-(J17-Pin_4-Pad4)
- J18 pad 4: GND -> EXT_I2C_SCL
- J19 pad 4: GND -> unconnected-(J19-Pin_4-Pad4)
- J20 pad 1: +3.3V -> +5V
- J21 pad 1: +3.3V -> +5V
Routing:
- net +5V: track 116.4 -> 240.7 mm, vias 1 -> 5
- net EXT_I2C_SDA: track 79.2 -> 142.5 mm, vias 1 -> 4
- net EXT_I2C_SCL: track 78.0 -> 131.6 mm, vias 1 -> 3
- net GND: track 272.3 -> 238.9 mm
- net +3.3V: track 420.3 -> 399.6 mm
- net /MCU/SWDIO: track 70.0 -> 65.3 mm, vias 2 -> 3
- net BUZZER_LOW: track 15.9 -> 18.2 mm
- net TELEM_RX: track 45.3 -> 43.4 mm, vias 1 -> 2
- net GPS_TX: track 43.8 -> 42.4 mm, vias 1 -> 2
- net TELEM_TX: track 42.8 -> 41.4 mm, vias 1 -> 2
- net NRST: track 65.2 -> 64.1 mm
- net RC_TX: track 30.1 -> 29.2 mm, vias 1 -> 2
- net GPS_RX: track 45.8 -> 45.3 mm, vias 1 -> 2
- net /MCU/SWCLK: track 55.5 -> 56.0 mm, vias 1 -> 2
