File: interfaces.kicad_sch (KiCad schematic)
At the start: 63 parts, among them J10 Conn_01x03, J11 Conn_01x03, J12 Conn_01x03, J13 Conn_01x03, J14 Conn_01x03, J15 Conn_01x03, J16 Conn_01x03, J17 RC_USART2_3V3_LOGIC, J18 GPS, J19 TELEMETRY, J20 COMPASS_I2C4_3V3, J21 AIRSPEED_I2C4_3V3, J22 SERVO_BEC_6V_INPUT, J23 BATTERY_SENSE_ONLY, J24 ACTIVE_BUZZER_5V_20mA_MAX, J5 Conn_01x03, J6 Conn_01x03, J7 Conn_01x03, J8 Conn_01x03, J9 Conn_01x03, Q1 MMBT3904, SW1 RESET, SW2 SAFETY, U9 USBLC6-2SC6

Commit message: Update JST-GH interfaces and add board 3D preview
Parts:
- J17: value RC_USART2_3V3_LOGIC -> RC_UART_GH6_NO_FLOW; footprint Connector_PinHeader_2.54mm:PinHeader_1x04_P2.54mm_Vertical -> Connector_JST:JST_GH_SM06B-GHS-TB_1x06-1MP_P1.25mm_Horizontal; symbol Connector_Generic:Conn_01x04 -> Connector_Generic:Conn_01x06
- J18: value GPS -> GPS_PIXHAWK_GPS2; footprint Connector_PinHeader_2.54mm:PinHeader_1x04_P2.54mm_Vertical -> Connector_JST:JST_GH_SM06B-GHS-TB_1x06-1MP_P1.25mm_Horizontal; symbol Connector_Generic:Conn_01x04 -> Connector_Generic:Conn_01x06
- J19: value TELEMETRY -> TELEM_GH6_NO_FLOW; footprint Connector_PinHeader_2.54mm:PinHeader_1x04_P2.54mm_Vertical -> Connector_JST:JST_GH_SM06B-GHS-TB_1x06-1MP_P1.25mm_Horizontal; symbol Connector_Generic:Conn_01x04 -> Connector_Generic:Conn_01x06
- J20: value COMPASS_I2C4_3V3 -> COMPASS_I2C4_5V; footprint Connector_PinHeader_2.54mm:PinHeader_1x04_P2.54mm_Vertical -> Connector_JST:JST_GH_SM04B-GHS-TB_1x04-1MP_P1.25mm_Horizontal
- J21: value AIRSPEED_I2C4_3V3 -> AIRSPEED_I2C4_5V; footprint Connector_PinHeader_2.54mm:PinHeader_1x04_P2.54mm_Vertical -> Connector_JST:JST_GH_SM04B-GHS-TB_1x04-1MP_P1.25mm_Horizontal
- J24: value ACTIVE_BUZZER_5V_20mA_MAX -> BUZZER_5V_20mA_MAX; footprint Connector_PinHeader_2.54mm:PinHeader_1x02_P2.54mm_Vertical -> Connector_JST:JST_GH_SM02B-GHS-TB_1x02-1MP_P1.25mm_Horizontal
Connections:
- net +3.3V: no longer J20.1 (Pin_1), J21.1 (Pin_1)
- net +5V: now also J20.1 (Pin_1), J21.1 (Pin_1)
- net EXT_I2C_SCL: now also J18.4 (Pin_4)
- net EXT_I2C_SDA: now also J18.5 (Pin_5)
- net GND: now also J17.6 (Pin_6), J18.6 (Pin_6), J19.6 (Pin_6); no longer J17.4 (Pin_4), J18.4 (Pin_4), J19.4 (Pin_4)
- no-connect marks 6 -> 10
