File: untitled.kicad_sch (KiCad schematic)
At the start: 55 parts, among them J1 Conn_01x05_Pin, J2 USB_C_Receptacle_USB2.0_14P, J3 Micro_SD_Card, U1 STM32H743VITx, U2 ICM-42688-P, U3 ICM-42688-P, U4 BMI088, U5 MB85RS64, U6 BMP390, U7 BMP390, Y1 8MHz

Commit message: Update JST-GH interfaces and add board 3D preview
Parts:
- J1: value Conn_01x05_Pin -> SWD_CUSTOM_GH5; footprint Connector_PinHeader_2.54mm:PinHeader_1x05_P2.54mm_Vertical -> Connector_JST:JST_GH_SM05B-GHS-TB_1x05-1MP_P1.25mm_Horizontal
